File: CatchTheLightV2.0.brd (EAGLE design)
At the start: 45 x 100 mm, 44 parts, among them J1 TC2030-IDC-NL, U1 ATMEGA328PB-ANR

Commit message: UMD Logo Added
Snazzy
Routing:
- net QTOUCH: vias 1 -> 0
Other:
- board text added: "Catch The Light V2"
- board text added: "Rev: E"
- board text removed: "Rev: D"
